File: kicad/Q1LMCKbdTester/Q1LMCKbdTester.kicad_sch (KiCad schematic)
At the start: 35 parts, among them J1 Conn_02x17_Odd_Even, J2 Conn_02x17_Odd_Even, J3 KB, J4 Wrap, J5 Barrel_Jack_Switch, U1 STM32F411 BlackPill, U2 L7805, U3 L7812, U4 L7905, U5 L7912

Commit message: Now sent to jlcpcb..
Parts:
- added H1, H2, H3, H4: MountingHole, MountingHole:MountingHole_3.2mm_M3_DIN965, symbol Mechanical:MountingHole
- added HS1: Heatsink_Pad_2Pin, Heatsink:Heatsink_Fischer_SK104-STCB_35x13mm__2xDrill3.5mm_ScrewM3, symbol Mechanical:Heatsink_Pad_2Pin
- C1: footprint (none) -> Capacitor_THT:CP_Radial_D10.0mm_P5.00mm
- C2: footprint (none) -> Capacitor_THT:CP_Radial_D7.5mm_P2.50mm
- C3: renamed from C6; footprint (none) -> Capacitor_THT:CP_Radial_D7.5mm_P2.50mm
- C4: renamed from C5; footprint (none) -> Capacitor_THT:CP_Radial_D7.5mm_P2.50mm
- C5: renamed from C3; footprint (none) -> Capacitor_THT:CP_Radial_D7.5mm_P2.50mm
- C6: renamed from C4; footprint (none) -> Capacitor_THT:CP_Radial_D7.5mm_P2.50mm
- D1, D2, D3: footprint (none) -> Diode_THT:D_DO-41_SOD81_P10.16mm_Horizontal
- D10, D11, D4, D5, D6, D7, D8, D9: footprint (none) -> LED_THT:LED_D5.0mm
- J1: renamed from J5; footprint (none) -> Connector_BarrelJack:BarrelJack_Kycon_KLDX-0202-xC_Horizontal
- J2: renamed from J3; footprint (none) -> Connector_IDC:IDC-Header_2x17_P2.54mm_Vertical
- J3: renamed from J4; footprint (none) -> Connector_PinHeader_2.54mm:PinHeader_2x17_P2.54mm_Vertical
- J4: renamed from J1; value Conn_02x17_Odd_Even -> Wrap; footprint (none) -> Connector_PinHeader_2.54mm:PinHeader_2x17_P2.54mm_Vertical
- J5: renamed from J2; value Conn_02x17_Odd_Even -> OtherKB; footprint (none) -> Connector_IDC:IDC-Header_2x17_P2.54mm_Vertical
- R1, R2, R3, R4, R5, R6, R7, R8: footprint (none) -> Resistor_THT:R_Axial_DIN0207_L6.3mm_D2.5mm_P10.16mm_Horizontal
- U1: footprint (none) -> Package_DIP:DIP-40_W15.24mm
- U2: renamed from U5; footprint (none) -> Package_TO_SOT_THT:TO-220-3_Vertical
- U3: renamed from U4; footprint (none) -> Package_TO_SOT_THT:TO-220-3_Vertical
- U4: renamed from U2; footprint (none) -> Package_TO_SOT_THT:TO-220-3_Vertical
- U5: renamed from U3; footprint (none) -> Package_TO_SOT_THT:TO-220-3_Vertical
Connections:
- no-connect marks 22 -> 24
